File: Circuit/OpeNITHM.kicad_pcb (KiCad board)
At the start: 2 copper layers, 100 x 45.3 mm, 59 parts, among them J1 Conn_01x12, J2 Conn_01x12, J3 Conn_01x08, J4 Conn_01x11, J5 Conn_01x08, J6 Conn_01x11, J7 Conn_01x04

Commit message: Fix schematic files
Parts:
- removed TP27: Guard, Connector_Wire:SolderWirePad_1x01_Drill1mm
- added G***: LOGO, OpeNITHM:OpeNITHM, F.Cu at (155.0, 80.5)
- added REF**: PinSocket_1x11_P2.54mm_Vertical, Connector_PinSocket_2.54mm:PinSocket_1x11_P2.54mm_Vertical, F.Cu at (195.6, 59.7)
- added REF**: MountingHole_2.2mm_M2, MountingHole:MountingHole_2.2mm_M2, F.Cu at (201.9, 50.8)
- added REF**: MountingHole_2.2mm_M2, MountingHole:MountingHole_2.2mm_M2, F.Cu at (201.9, 85.1)
- added REF**: MountingHole_2.2mm_M2, MountingHole:MountingHole_2.2mm_M2, F.Cu at (108.0, 85.1)
- added REF**: PinSocket_1x11_P2.54mm_Vertical, Connector_PinSocket_2.54mm:PinSocket_1x11_P2.54mm_Vertical, F.Cu at (139.7, 59.7)
- added REF**: MountingHole_2.2mm_M2, MountingHole:MountingHole_2.2mm_M2, F.Cu at (108.0, 50.8)
Routing:
- net /SEND: track 47.8 -> 35.3 mm
Other:
- board text removed: "Guard"

Commit message: Add GUARD pads and silk for RGB LED strip connector
Parts:
- added TP9: TestPoint, Connector_Wire:SolderWirePad_1x01_Drill1mm_Diameter2mm, F.Cu at (171.4, 86.4)
- added TP9: TestPoint, Connector_Wire:SolderWirePad_1x01_Drill1mm_Diameter2mm, F.Cu at (138.4, 86.4)
Other:
- board text added: "GUARD"
Changed lines of the file:
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@@
   (general
     (thickness 1.6)
-    (drawings 72)
+    (drawings 85)
     (tracks 306)
     (zones 0)
-    (modules 65)
+    (modules 67)
     (nets 42)
   )
@@
     (mod_text_width 0.15)
     (pad_size 2 2)
-    (pad_drill 0.8001)
+    (pad_drill 1)
     (pad_to_mask_clearance 0.051)
     (solder_mask_min_width 0.25)
@@
     (visible_elements 7FFFFFFF)
     (pcbplotparams
-      (layerselection 0x010fc_ffffffff)
+      (layerselection 0x010f0_ffffffff)
       (usegerberextensions false)
       (usegerberattributes false)
@@
       (outputformat 1)
       (mirror false)
-      (drillshape 1)
+      (drillshape 0)
       (scaleselection 1)
-      (outputdirectory ""))
+      (outputdirectory "New folder/"))
   )
   (net 0 "")
@@
     (add_net "Net-(R19-Pad1)")
   )
+  (module Connector_Wire:SolderWirePad_1x01_Drill1mm_Diameter2mm (layer F.Cu)
+    (at 171.45 86.36)
+    (descr "Wire solder connection")
+    (tags connector)
+    (attr virtual)
+    (fp_text reference TP9 (at 0 -3.81) (layer F.SilkS) hide
+      (effects (font (size 1 1) (thickness 0.15)))
+    )
+    (fp_text value TestPoint (at 0 3.175) (layer F.Fab)
+      (effects (font (size 1 1) (thickness 0.15)))
+    )
+    (fp_line (start 1.75 1.75) (end -1.75 1.75) (layer F.CrtYd) (width 0.05))
+    (fp_line (start 1.75 1.75) (end 1.75 -1.75) (layer F.CrtYd) (width 0.05))
+    (fp_line (start -1.75 -1.75) (end -1.75 1.75) (layer F.CrtYd) (width 0.05))
+    (fp_line (start -1.75 -1.75) (end 1.75 -1.75) (layer F.CrtYd) (width 0.05))
+    (fp_text user %R (at 0 0) (layer F.Fab)
+      (effects (font (size 1 1) (thickness 0.15)))
+    )
+    (pad 1 thru_hole circle (at 0 0) (size 2 2) (drill 1) (layers *.Cu *.Mask)
+      (net 17 /SEND))
+  )
+  (module Connector_Wire:SolderWirePad_1x01_Drill1mm_Diameter2mm (layer F.Cu)
+    (at 138.43 86.36)
+    (descr "Wire solder connection")
+    (tags connector)
+    (attr virtual)
+    (fp_text reference TP9 (at 0 -3.81) (layer F.SilkS) hide
+      (effects (font (size 1 1) (thickness 0.15)))
+    )
+    (fp_text value TestPoint (at 0 3.175) (layer F.Fab)
+      (effects (font (size 1 1) (thickness 0.15)))
+    )
+    (fp_text user %R (at 0 0) (layer F.Fab)
+      (effects (font (size 1 1) (thickness 0.15)))
+    )
+    (fp_line (start -1.75 -1.75) (end 1.75 -1.75) (layer F.CrtYd) (width 0.05))
+    (fp_line (start -1.75 -1.75) (end -1.75 1.75) (layer F.CrtYd) (width 0.05))
+    (fp_line (start 1.75 1.75) (end 1.75 -1.75) (layer F.CrtYd) (width 0.05))
+    (fp_line (start 1.75 1.75) (end -1.75 1.75) (layer F.CrtYd) (width 0.05))
+    (pad 1 thru_hole circle (at 0 0) (size 2 2) (drill 1) (layers *.Cu *.Mask)
+      (net 17 /SEND))
+  )
   (module Connector_PinSocket_2.54mm:PinSocket_1x11_P2.54mm_Vertical (layer F.Cu)
     (at 195.58 59.69 270)
@@
     (descr "Through hole straight socket strip, 1x04, 2.54mm pitch, single row (from Kicad 4.0.7), script generated")
     (tags "Through hole socket strip THT 1x04 2.54mm single row")
-    (fp_text reference J7 (at 0 -2.54 180) (layer F.SilkS)
+    (fp_text reference J7 (at 0 -2.6 180) (layer F.SilkS)
       (effects (font (size 1 1) (thickness 0.15)))
     )
@@
       (xy 0.543463 -1.067512)) (layer F.SilkS) (width 0.01))
   )
-  (gr_text "PCB by mickabrig7" (at 165 83.5) (layer F.SilkS)
+  (gr_line (start 149.098 84.836) (end 149.606 84.836) (layer F.SilkS) (width 0.3))
+  (gr_line (start 149.606 84.328) (end 149.098 84.836) (layer F.SilkS) (width 0.3))
+  (gr_line (start 149.606 84.836) (end 149.606 84.328) (layer F.SilkS) (width 0.3))
+  (gr_text GUARD (at 170.815 84.25) (layer F.SilkS)
+    (effects (font (size 0.7 0.7) (thickness 0.175)))
+  )
+  (gr_line (start 172.72 85.09) (end 172.72 84.455) (layer F.SilkS) (width 0.2))
+  (gr_line (start 172.72 83.82) (end 172.72 83.185) (layer F.SilkS) (width 0.2))
+  (gr_line (start 172.72 86.36) (end 172.72 85.725) (layer F.SilkS) (width 0.2))
+  (gr_line (start 172.72 87.63) (end 172.72 86.995) (layer F.SilkS) (width 0.2))
+  (gr_line (start 137.16 83.82) (end 137.16 83.185) (layer F.SilkS) (width 0.2))
+  (gr_text GUARD (at 139.065 84.25) (layer F.SilkS)
+    (effects (font (size 0.7 0.7) (thickness 0.175)))
+  )
+  (gr_line (start 137.16 86.36) (end 137.16 85.725) (layer F.SilkS) (width 0.2))
+  (gr_line (start 137.16 87.63) (end 137.16 86.995) (layer F.SilkS) (width 0.2))
+  (gr_line (start 137.16 85.09) (end 137.16 84.455) (layer F.SilkS) (width 0.2))
+  (gr_line (start 140.97 88) (end 140.97 83) (layer F.SilkS) (width 0.2))
+  (gr_text "PCB by\nmickabrig7" (at 165.1 83.82) (layer F.SilkS)
     (effects (font (size 0.7 0.7) (thickness 0.125)))
   )
@@
   (gr_circle (center 107.95 85.09) (end 109.65 85.09) (layer B.SilkS) (width 1))
   (gr_circle (center 107.95 50.8) (end 109.65 50.8) (layer B.SilkS) (width 1))
-  (gr_text "Design by WinEpic" (at 145 83.5) (layer F.SilkS)
+  (gr_text "Design by\nWinEpic" (at 144.78 83.82) (layer F.SilkS)
     (effects (font (size 0.7 0.7) (thickness 0.125)))
   )
@@
   (gr_line (start 205 62.92) (end 200 62.92) (layer F.SilkS) (width 0.2))
   (gr_line (start 205 73.08) (end 200 73.08) (layer F.SilkS) (width 0.2))
-  (gr_line (start 171.45 88) (end 171.45 83) (layer F.SilkS) (width 0.2))
+  (gr_line (start 168.91 88) (end 168.91 83) (layer F.SilkS) (width 0.2))
   (gr_line (start 194.31 88) (end 194.31 83) (layer F.SilkS) (width 0.2))
-  (gr_line (start 171.45 83) (end 194.31 83) (layer F.SilkS) (width 0.2))
-  (gr_line (start 115.57 83) (end 138.43 83) (layer F.SilkS) (width 0.2))
+  (gr_line (start 168.91 83) (end 194.31 83) (layer F.SilkS) (width 0.2))
+  (gr_line (start 115.57 83) (end 140.97 83) (layer F.SilkS) (width 0.2))
   (gr_line (start 115.57 88) (end 115.57 83) (layer F.SilkS) (width 0.2))
-  (gr_line (start 138.43 88) (end 138.43 83) (layer F.SilkS) (width 0.2))
   (gr_line (start 110 57.84) (end 110 78.16) (layer F.SilkS) (width 0.2))
   (gr_line (start 105 78.16) (end 110 78.16) (layer F.SilkS) (width 0.2))
