File: Circuit-Teensy/OpeNITHM.kicad_pcb (KiCad board)
At the start: 2 copper layers, 100 x 45.3 mm, 26 parts, among them J1 Conn_01x14, J10 Conn_01x11, J11 Conn_01x11, J2 Conn_01x14, J3 Conn_01x08, J4 Conn_01x11, J5 Conn_01x08, J6 Conn_01x11, J7 Conn_02x08_Odd_Even, J8 Conn_02x08_Odd_Even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

Commit message: Updated main OpeNITHM board to v1.1
Code has not been updated yet, do not use
Parts:
- R17, R18, R19: value 100 -> 33; footprint Resistor_THT:R_Axial_DIN0204_L3.6mm_D1.6mm_P5.08mm_Horizontal -> Resistor_THT:R_Axial_DIN0207_L6.3mm_D2.5mm_P7.62mm_Horizontal
- R20, R21, R22, R23, R24, R25: value 10k -> 51k
- moved R17 4.32 mm to (193.8, 50.5)
- moved R18 2.79 mm to (183.6, 49.3)
- moved R19 1.27 mm to (173.5, 47.8)
Connections:
- J1 pad 10: /AIR_4 -> Net-(J1-Pad10)
- J1 pad 11: /AIR_5 -> Net-(J1-Pad11)
- J1 pad 12: /AIR_0 -> Net-(J1-Pad12)
- J1 pad 13: /AIR_1 -> /RGB_DO
- J1 pad 14: /AIR_2 -> Net-(J1-Pad14)
- J1 pad 2: Net-(J1-Pad2) -> /MUX_2
- J1 pad 3: Net-(J1-Pad3) -> /MUX_1
- J1 pad 4: Net-(J1-Pad4) -> /MUX_0
- J1 pad 5: Net-(J1-Pad5) -> /TOUCH_1
- J1 pad 6: /RGB_DO -> Net-(J1-Pad6)
- J1 pad 8: /AIR_3 -> /LED_1
- J1 pad 9: /RGB_DO -> /LED_0
- J2 pad 11: /LED_0 -> /TOUCH_0
- J2 pad 4: /TOUCH_1 -> /AIR_3
- J2 pad 5: /TOUCH_0 -> /AIR_4
- J2 pad 6: /LED_1 -> /AIR_5
- J2 pad 7: /MUX_0 -> /AIR_0
- J2 pad 8: /MUX_1 -> /AIR_1
- J2 pad 9: /MUX_2 -> /AIR_2
- J8 pad 16: Net-(J8-Pad16) -> GND
Routing:
- net /LED_1: track 23.4 -> 43.8 mm
- net /TOUCH_1: track 32.3 -> 16.0 mm
- net /AIR_1: track 57.5 -> 73.1 mm
- net /AIR_0: track 54.9 -> 70.2 mm
- net /AIR_2: track 60.2 -> 75.2 mm
- net /AIR_3: track 72.3 -> 85.4 mm
- net /MUX_1: track 77.2 -> 64.3 mm, vias 2 -> 1
- net /MUX_0: track 72.8 -> 60.0 mm, vias 2 -> 1
- net /LED_0: track 43.1 -> 55.0 mm
- net /MUX_2: track 82.4 -> 72.2 mm, vias 2 -> 1
- net /AIR_5: track 73.4 -> 83.0 mm
- net /AIR_4: track 74.8 -> 84.1 mm
- net /RGB_DO: track 50.9 -> 44.9 mm
- net GND: track 5.08 -> 0.00 mm
- net /LED_2: track 36.6 -> 32.3 mm
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Other:
- board text added: "v1.1"
